Commit message: Assets: Updated walls of robot | Description: Updated macro for colors

File: orion_description/urdf/include/orion_arms.urdf.xacro (robot description, xacro)
@@ -12,5 +12,16 @@
                     scale="0.001 0.001 0.001"/>
                 </geometry>
-                <material name="PLAWhite"/>
+                <xacro:if value="${color == 'mdf'}">
+                    <material name="MDF"/>
+                </xacro:if>
+                <xacro:if value="${color == 'transparent'}">
+                    <material name="TransparentBlack"/>
+                </xacro:if>
+                <xacro:if value="${color == 'pla'}">
+                    <material name="PLAWhite"/>
+                </xacro:if>
+                <xacro:if value="${color == 'gold'}">
+                    <material name="Gold"/>
+                </xacro:if>
             </visual>
             <collision>

File: orion_description/urdf/include/orion_base.urdf.xacro (robot description, xacro)
@@ -76,4 +76,7 @@
                     <material name="PLAWhite"/>
                 </xacro:if>
+                <xacro:if value="${color == 'gold'}">
+                    <material name="Gold"/>
+                </xacro:if>
         </visual>
         <collision>
@@ -127,4 +130,7 @@
                 <xacro:if value="${color == 'pla'}">
                     <material name="PLAWhite"/>
+                </xacro:if>
+                <xacro:if value="${color == 'gold'}">
+                    <material name="Gold"/>
                 </xacro:if>
         </visual>
@@ -743,12 +749,15 @@
         </geometry>
         <xacro:if value="${color == 'mdf'}">
-                <material name="MDF"/>
-            </xacro:if>
-            <xacro:if value="${color == 'transparent'}">
-                <material name="TransparentBlack"/>
-            </xacro:if>
-            <xacro:if value="${color == 'pla'}">
-                <material name="PLAWhite"/>
-            </xacro:if>
+            <material name="MDF"/>
+        </xacro:if>
+        <xacro:if value="${color == 'transparent'}">
+            <material name="TransparentBlack"/>
+        </xacro:if>
+        <xacro:if value="${color == 'pla'}">
+            <material name="PLAWhite"/>
+        </xacro:if>
+        <xacro:if value="${color == 'gold'}">
+            <material name="Gold"/>
+        </xacro:if>
     </visual>
     <collision>

File: orion_description/urdf/include/orion_macros.urdf.xacro (robot description, xacro)
@@ -95,4 +95,7 @@
                 <material name="PLAWhite"/>
             </xacro:if>
+            <xacro:if value="${color == 'gold'}">
+                <material name="Gold"/>
+            </xacro:if>
         </visual>
         <collision>
@@ -754,4 +757,7 @@
                 <material name="PLAWhite"/>
             </xacro:if>
+            <xacro:if value="${color == 'gold'}">
+                <material name="Gold"/>
+            </xacro:if>
         </visual>
         <collision>
@@ -804,4 +810,7 @@
             <xacro:if value="${color == 'pla'}">
                 <material name="PLAWhite"/>
+            </xacro:if>
+            <xacro:if value="${color == 'gold'}">
+                <material name="Gold"/>
             </xacro:if>
         </visual>
@@ -1004,5 +1013,16 @@
                     scale="0.001 0.001 0.001"/>
                 </geometry>
-                <material name="PLAWhite"/>
+                <xacro:if value="${color == 'mdf'}">
+                    <material name="MDF"/>
+                </xacro:if>
+                <xacro:if value="${color == 'transparent'}">
+                    <material name="TransparentBlack"/>
+                </xacro:if>
+                <xacro:if value="${color == 'pla'}">
+                    <material name="PLAWhite"/>
+                </xacro:if>
+                <xacro:if value="${color == 'gold'}">
+                    <material name="Gold"/>
+                </xacro:if>
             </visual>
             <collision>

File: orion_description/urdf/include/orion_materials.urdf.xacro (robot description, xacro)
@@ -30,4 +30,8 @@
         <color rgba="0.71 0.65 0.26 1.0"/>
     </material>
+    <!-- Equivalent to RGB(293, 191, 4) -->
+    <material name="Gold">
+        <color rgba="0.71 0.65 0.26 1.0"/>
+    </material>
     <!-- Equivalent to RGB(128, 128, 128) -->
     <material name="MetalGray">

Commit message: Description: Improving URDF notes and fixing typos

File: orion_description/urdf/include/orion_arms.urdf.xacro (robot description, xacro)
@@ -1,8 +1,9 @@
 <?xml version="1.0"?>
+<!-- @file orion_arms.urdf.xacro
+     @brief Simple arm link definitions attached to the servo connectors. -->
 <robot xmlns:xacro="http://www.ros.org/wiki/xacro">
-<!-- This xacro file aims for adding the arms to the robot-->
     <xacro:if value="${servo}">
         <xacro:macro name="simple_arm" params="x y z parent side">
-            <!-- Link Spacer -->
+            <!-- Arm link -->
             <link name="simple_arm_${side}">
             <visual>
@@ -34,5 +35,5 @@
             <inertial>
                 <origin xyz="0.0 0.0 0.0" rpy="${-pi_2} 0.0 0.0"/>
-                <mass value="1"/>
+                <mass value="0.020"/>
                 <inertia ixx="8.550666163126637e-09" ixy="0" ixz="0"
                         iyy="8.960721799390997e-09" iyz="0"
@@ -40,5 +41,5 @@
             </inertial>
             </link>
-            <!-- Joint Spacer -->
+            <!-- Arm joint -->
             <joint name="simple_arm_${side}_joint" type="fixed">
                 <parent link="${parent}"/>
@@ -46,5 +47,5 @@
                 <origin xyz="${x} ${y} ${z}" rpy="0 0 0"/>
             </joint>
-            <!-- Gazebo Spacer -->
+            <!-- Gazebo properties -->
             <xacro:if value="${gazebo}">
                 <gazebo reference="simple_arm_${side}">

File: orion_description/urdf/include/orion_base.urdf.xacro (robot description, xacro)
@@ -1,5 +1,7 @@
 <?xml version="1.0"?>
+<!-- @file orion_base.urdf.xacro
+     @brief Mobile platform definition for ORION: base links, levels, spacers,
+     drive motors, caster wheel, floor components, sensors, and walls. -->
 <robot xmlns:xacro="http://www.ros.org/wiki/xacro">
-    <!-- This xacro file aims for adding the mobile platform to the robot-->
     <!-- ////////////////////////// BASE LINK //////////////////////////////-->
     <link name="base_link"/>
@@ -12,6 +14,6 @@
     </joint>
     <!-- ///////////////////////// PROPERTIES //////////////////////////////-->
-    <xacro:property name="level_height" value="0.08"/>
-    <xacro:property name="thickness" value="0.0025"/>
+    <xacro:property name="level_height" value="0.08"/>   <!-- m: vertical distance between platform levels -->
+    <xacro:property name="thickness" value="0.0025"/>    <!-- m: platform panel thickness -->
     <!-- /////////////////////////// LEVELS ///////////////////////////////-->
     <xacro:com_base level="0" parent="middle_base" x="0" y="0"
@@ -505,5 +507,5 @@
     <xacro:complete_front_wall id="flidar" parent="base_l1_s2" front="2"
         x="${0.115/2}" z="${0.082/2 + 0.0025/2}" level="1"/>
-    <!-- ////////////////// THIRD FLOOR COMPONENTES ////////////////////// -->
+    <!-- ////////////////// THIRD FLOOR COMPONENTS ////////////////////// -->
     <xacro:if value="${rasp == 'rpi4'}">
         <xacro:speakers_mount parent="base_l2_s2" front="2" side="1" x="-0.0025"
@@ -567,9 +569,9 @@
             x="${0.115/2}" z="${0.082/2 + 0.0025/2}" level="2"/>
     </xacro:if>
-    <!-- ////////////////// FOURTH FLOOR COMPONENTES ////////////////////// -->
+    <!-- ////////////////// FOURTH FLOOR COMPONENTS ////////////////////// -->
     <xacro:unless value="${simplified}">
         <xacro:x4xmetric_spacer id="m3x10" element="${rasp}" parent="base_l3_s2"
         offset_x="${0.049/2}" offset_y="${0.058/2}" x="0" y="0.0435" z="0.0025"/>
-        <!-- Link Rasberry Pi -->
+        <!-- Link Raspberry Pi -->
         <link name="${rasp}">
             <visual>
@@ -698,5 +700,5 @@
         </joint>
         <xacro:if value="${gazebo}">
-            <gazebo reference="esp32_adapter">
+            <gazebo reference="esp32_2_adapter">
                 <mu1>1.0</mu1>
                 <mu2>1.0</mu2>
@@ -734,5 +736,5 @@
         </joint>
         <xacro:if value="${gazebo}">
-            <gazebo reference="esp32">
+            <gazebo reference="esp32_2">
                 <mu1>1.0</mu1>
                 <mu2>1.0</mu2>

File: orion_description/urdf/include/orion_cameras.urdf.xacro (robot description, xacro)
@@ -1,4 +1,7 @@
 <?xml version="1.0"?>
+<!-- @file orion_cameras.urdf.xacro
+     @brief Camera link definitions for ORION: Astra S, OS30A, and MaixSense A010. -->
 <robot xmlns:xacro="http://www.ros.org/wiki/xacro">
+    <!-- Mounting level for cameras: level 2, side 1 (third platform from base) -->
     <xacro:property name="level_cam" value="base_l2_s1"/>
     <!--  //////////////////////// ASTRA_S CAM ///////////////////////////// -->

File: orion_description/urdf/include/orion_macros.urdf.xacro (robot description, xacro)
@@ -1,3 +1,7 @@
 <?xml version="1.0"?>
+<!-- @file orion_macros.urdf.xacro
+     @brief Reusable xacro macros for ORION structural, mechanical, and sensor links.
+     Defines macros for spacers, platforms, drive motors, caster wheels, batteries,
+     servos, speakers, walls, metric spacers, touch sensors, and camera frames. -->
 <robot xmlns:xacro="http://www.ros.org/wiki/xacro">
     <!--//////////////////// MATH AND NUMS MACROS ///////////////////////-->
@@ -119,8 +123,10 @@
             <origin xyz="${x + (mul*0.115/2)} ${y} ${z}" rpy="0 0 0"/>
         </joint>
+        <xacro:if value="${gazebo}">
         <gazebo reference="base_l${level}_s${side}">
             <mu1>1.0</mu1>
             <mu2>1.0</mu2>
         </gazebo>
+        </xacro:if>
     </xacro:macro>
     <!-- ...................... Complete base ............................ -->
@@ -490,5 +496,5 @@
     </xacro:macro>
     <!-- ........................ Battery holder macro ........................ -->
-    <xacro:macro name="bat_hold" params=" parent element num x y z">
+    <xacro:macro name="bat_hold" params="parent element num x y z">
         <!-- Link -->
         <link name="${element}_${num}">

File: orion_description/urdf/include/orion_materials.urdf.xacro (robot description, xacro)
@@ -1,5 +1,6 @@
 <?xml version="1.0"?>
+<!-- @file orion_materials.urdf.xacro
+     @brief Material and color definitions used across the ORION URDF. -->
 <robot xmlns:xacro="http://www.ros.org/wiki/xacro">
-<!-- This xacro file aims for defining materials and color properties for the URDF-->
     <!-- Equivalent to RGB(0, 79, 148) -->
     <material name="ArduinoBlue">
@@ -30,7 +31,7 @@
         <color rgba="0.71 0.65 0.26 1.0"/>
     </material>
-    <!-- Equivalent to RGB(293, 191, 4) -->
+    <!-- Equivalent to RGB(212, 173, 54) -->
     <material name="Gold">
-        <color rgba="0.71 0.65 0.26 1.0"/>
+        <color rgba="0.83 0.68 0.21 1.0"/>
     </material>
     <!-- Equivalent to RGB(128, 128, 128) -->

File: orion_description/urdf/include/orion_ros2_control.urdf.xacro (robot description, xacro)
@@ -1,3 +1,6 @@
 <?xml version="1.0"?>
+<!-- @file orion_ros2_control.urdf.xacro
+     @brief ros2_control hardware interface tags for ORION differential drive and servo arms.
+     Exposes DiffDriveOrion and ForwardOrion plugins to the controller manager. -->
 <robot xmlns:xacro="http://www.ros.org/wiki/xacro">
     <xacro:if value="${ros2_control}">
@@ -18,4 +21,7 @@
                     </xacro:if>
                 </hardware>
+                <!-- NOTE: command interface limits (~26.7 RPM) are conservative vs
+                     physical joint limits (10.47 rad/s for 100 RPM motors).
+                     Review against mobile_base_controller.yaml if updating motor specs. -->
                 <joint name="coupling_11_joint">
                     <command_interface name="velocity">

File: orion_description/urdf/orion.urdf.xacro (robot description, xacro)
@@ -1,3 +1,8 @@
 <?xml version="1.0"?>
+<!-- @file orion.urdf.xacro
+     @brief Top-level robot description for ORION. Declares all configurable
+     properties (camera, servo, rasp, motor, ctl_type, etc.) and includes
+     the modular xacro files for materials, macros, base, arms, cameras,
+     and ros2_control tags. -->
 <robot xmlns:xacro="http://www.ros.org/wiki/xacro" name="orion">
     <xacro:property name="camera" default="$(arg camera)"/>
