Commit message: Description: Replacing color and gz friction with macros, clearning macro files and updating comments

File: orion_description/urdf/include/orion_arms.urdf.xacro (robot description, xacro)
@@ -13,16 +13,5 @@
                     scale="0.001 0.001 0.001"/>
                 </geometry>
-                <xacro:if value="${color == 'mdf'}">
-                    <material name="MDF"/>
-                </xacro:if>
-                <xacro:if value="${color == 'transparent'}">
-                    <material name="TransparentBlack"/>
-                </xacro:if>
-                <xacro:if value="${color == 'pla'}">
-                    <material name="PLAWhite"/>
-                </xacro:if>
-                <xacro:if value="${color == 'gold'}">
-                    <material name="Gold"/>
-                </xacro:if>
+                <xacro:apply_color_material/>
             </visual>
             <collision>
@@ -47,11 +36,6 @@
                 <origin xyz="${x} ${y} ${z}" rpy="0 0 0"/>
             </joint>
-            <!-- Gazebo properties -->
-            <xacro:if value="${gazebo}">
-                <gazebo reference="simple_arm_${side}">
-                    <mu1>0.0005</mu1>
-                    <mu2>0.0005</mu2>
-                </gazebo>
-            </xacro:if>
+            <xacro:gazebo_friction link="simple_arm_${side}"
+                mu1="0.0005" mu2="0.0005"/>
         </xacro:macro>
         <xacro:simple_arm x="0" y="0" z="0.0045" parent="servo_conn_1" side="1"/>

File: orion_description/urdf/include/orion_base.urdf.xacro (robot description, xacro)
@@ -62,50 +62,6 @@
             z="0.0025"/>
         <!-- ..................... Battery Platform ....................... -->
-        <link name="bat_platform">
-        <visual>
-            <origin xyz="0 0 0" rpy="0 0 ${pi_2}"/>
-            <geometry>
-            <mesh filename="package://orion_description/meshes/bathold_support.stl"
-                scale="0.001 0.001 0.001"/>
-            </geometry>
-            <xacro:if value="${color == 'mdf'}">
-                    <material name="MDF"/>
-                </xacro:if>
-                <xacro:if value="${color == 'transparent'}">
-                    <material name="TransparentBlack"/>
-                </xacro:if>
-                <xacro:if value="${color == 'pla'}">
-                    <material name="PLAWhite"/>
-                </xacro:if>
-                <xacro:if value="${color == 'gold'}">
-                    <material name="Gold"/>
-                </xacro:if>
-        </visual>
-        <collision>
-            <origin xyz="0 0 0" rpy="0 0 ${pi_2}"/>
-            <geometry>
-            <mesh filename="package://orion_description/meshes/bathold_support.stl"
-                scale="0.001 0.001 0.001"/>
-            </geometry>
-        </collision>
-        <inertial>
-            <origin xyz="0 0 0" rpy="0 0 ${pi_2}"/>
-            <mass value="0.018"/>
-            <inertia ixx="1.2564374999999998e-05" ixy="0.0" ixz="0.0"
-                    iyy="2.6539499999999996e-05" iyz="0.0"
-                    izz="3.9091874999999996e-05"/>
-        </inertial>
-        </link>
-        <joint name="bat_platform_joint" type="fixed">
-            <parent link="base_l0_s1"/>
-            <child link="bat_platform"/>
-            <origin xyz="0.005 0 0.0125" rpy="0 0 0"/>
-        </joint>
-        <xacro:if value="${gazebo}">
-            <gazebo reference="bat_platform">
-                <mu1>1.0</mu1>
-                <mu2>1.0</mu2>
-            </gazebo>
-        </xacro:if>
+        <xacro:bat_platform_unit suffix="" parent="base_l0_s1"
+            x="0.005" y="0" z="0.0125"/>
         <!-- ....................... Battery Stacks ........................ -->
         <xacro:stack_bat parent="bat_platform" num="1" x="0" y="-0.023" z="0.0025"/>
@@ -117,50 +73,6 @@
             z="0.0175"/>
         <!-- ..................... Battery Platform ....................... -->
-        <link name="bat_platform_2">
-        <visual>
-            <origin xyz="0 0 0" rpy="0 0 ${pi_2}"/>
-            <geometry>
-            <mesh filename="package://orion_description/meshes/bathold_support.stl"
-                scale="0.001 0.001 0.001"/>
-            </geometry>
-            <xacro:if value="${color == 'mdf'}">
-                    <material name="MDF"/>
-                </xacro:if>
-                <xacro:if value="${color == 'transparent'}">
-                    <material name="TransparentBlack"/>
-                </xacro:if>
-                <xacro:if value="${color == 'pla'}">
-                    <material name="PLAWhite"/>
-                </xacro:if>
-                <xacro:if value="${color == 'gold'}">
-                    <material name="Gold"/>
-                </xacro:if>
-        </visual>
-        <collision>
-            <origin xyz="0 0 0" rpy="0 0 ${pi_2}"/>
-            <geometry>
-            <mesh filename="package://orion_description/meshes/bathold_support.stl"
-                scale="0.001 0.001 0.001"/>
-            </geometry>
-        </collision>
-        <inertial>
-            <origin xyz="0 0 0" rpy="0 0 ${pi_2}"/>
-            <mass value="0.018"/>
-            <inertia ixx="1.2564374999999998e-05" ixy="0.0" ixz="0.0"
-                    iyy="2.6539499999999996e-05" iyz="0.0"
-                    izz="3.9091874999999996e-05"/>
-        </inertial>
-        </link>
-        <joint name="bat_platform_2_joint" type="fixed">
-            <parent link="base_l0_s1"/>
-            <child link="bat_platform_2"/>
-            <origin xyz="0.005 0 0.0375" rpy="0 0 0"/>
-        </joint>
-        <xacro:if value="${gazebo}">
-            <gazebo reference="bat_platform_2">
-                <mu1>1.0</mu1>
-                <mu2>1.0</mu2>
-            </gazebo>
-        </xacro:if>
+        <xacro:bat_platform_unit suffix="_2" parent="base_l0_s1"
+            x="0.005" y="0" z="0.0375"/>
         <!-- ....................... Battery Stacks ........................ -->
         <xacro:stack_bat parent="bat_platform_2" num="3" x="0" y="-0.023" z="0.0025"/>
@@ -201,10 +113,5 @@
         <origin xyz="-0.023453 0.031351 0.0125" rpy="0 0 0"/>
     </joint>
-    <xacro:if value="${gazebo}">
-            <gazebo reference="driver">
-                <mu1>1.0</mu1>
-                <mu2>1.0</mu2>
-            </gazebo>
-        </xacro:if>
+    <xacro:gazebo_friction link="driver"/>
         <!-- ........................ Regulator Support ......................... -->
         <link name="reg_support">
@@ -237,10 +144,5 @@
             <origin xyz="-0.026 -0.0275 0.0025" rpy="0 0 0"/>
         </joint>
-        <xacro:if value="${gazebo}">
-            <gazebo reference="reg_support">
-                <mu1>1.0</mu1>
-                <mu2>1.0</mu2>
-            </gazebo>
-        </xacro:if>
+        <xacro:gazebo_friction link="reg_support"/>
         <!-- ....................... Regulator ............................... -->
         <link name="regulator">
@@ -273,10 +175,5 @@
             <origin xyz="-0.0025 0 ${0.06/2 -0.0025}" rpy="0 0 0"/>
         </joint>
-        <xacro:if value="${gazebo}">
-            <gazebo reference="regulator">
-                <mu1>1.0</mu1>
-                <mu2>1.0</mu2>
-            </gazebo>
-        </xacro:if>
+        <xacro:gazebo_friction link="regulator"/>
     </xacro:unless>
         <!-- ......................... Switch ........................... -->
@@ -310,10 +207,5 @@
         <origin xyz="0.035 0.074 -0.015" rpy="0 0 0"/>
     </joint>
-    <xacro:if value="${gazebo}">
-        <gazebo reference="switch">
-            <mu1>1.0</mu1>
-            <mu2>1.0</mu2>
-        </gazebo>
-    </xacro:if>
+    <xacro:gazebo_friction link="switch"/>
     <!-- ......................... Walls definitions ...................... -->
     <xacro:complete_lateral_wall id="servo" parent="base_l0_s1" side="1"
@@ -333,75 +225,9 @@
         offset_x="${0.0577/2}" offset_y="${0.0607/2}" x="0.004" y="0" z="-0.01"/>
         <!-- .......................... Esp32 Adapter ....................... -->
-        <link name="esp32_adapter">
-            <visual>
-                <origin xyz="0 0 0" rpy="${pi} 0 0"/>
-                <geometry>
-                    <mesh filename="package://orion_description/meshes/esp32_adp.stl"
-                    scale="0.001 0.001 0.001"/>
-                </geometry>
-                <material name="RaspberryGreen"/>
-            </visual>
-            <collision>
-                <origin xyz="0 0 0" rpy="${pi} 0 0"/>
-                <geometry>
-                    <mesh filename="package://orion_description/meshes/esp32_adp.stl"
-                    scale="0.001 0.001 0.001"/>
-                </geometry>
-            </collision>
-            <inertial>
-                <origin xyz="0 0 0" rpy="${pi} 0 0"/>
-                <mass value="0.030"/>
-                <inertia ixx="1.1184306270694732e-05" ixy="0.0" ixz="0.0"
-                iyy="1.021680627069473e-05" iyz="0.0"
-                izz="2.0812499999999994e-05"/>
-            </inertial>
-        </link>
-        <joint name="esp32_adapter_joint" type="fixed">
-            <parent link="base_l1_s2"/>
-            <child link="esp32_adapter"/>
-            <origin xyz="0.004 0 -0.01" rpy="0 0 0"/>
-        </joint>
-        <xacro:if value="${gazebo}">
-            <gazebo reference="esp32_adapter">
-                <mu1>1.0</mu1>
-                <mu2>1.0</mu2>
-            </gazebo>
-        </xacro:if>
+        <xacro:esp32_adapter_unit suffix="" parent="base_l1_s2"
+            rpy="${pi} 0 0" x="0.004" y="0" z="-0.01"/>
         <!-- ....................... ESP32 ....................................... -->
-        <link name="esp32">
-            <visual>
-                <origin xyz="0 0 0" rpy="${pi} 0 ${-pi_2}"/>
-                <geometry>
-                    <mesh filename="package://orion_description/meshes/esp32.stl"
-                    scale="0.001 0.001 0.001"/>
-                </geometry>
-                <material name="SoftBlack"/>
-            </visual>
-            <collision>
-                <origin xyz="0 0 0" rpy="${pi} 0 ${-pi_2}"/>
-                <geometry>
-                    <mesh filename="package://orion_description/meshes/esp32.stl"
-                    scale="0.001 0.001 0.001"/>
-                </geometry>
-            </collision>
-            <inertial>
-                <origin xyz="0 0 0" rpy="${pi} 0 ${-pi_2}"/>
-                <mass value="0.0201"/>
-                <inertia ixx="4.904162034278915e-06" ixy="0.0" ixz="0.0"
-                iyy="1.5830928543782435e-06" iyz="0.0"
-                izz="6.0040505352397235e-06"/>
-            </inertial>
-        </link>
-        <joint name="esp32_joint" type="fixed">
-            <parent link="esp32_adapter"/>
-            <child link="esp32"/>
-            <origin xyz="0.002 0 -0.01" rpy="0 0 0"/>
-        </joint>
-        <xacro:if value="${gazebo}">
-            <gazebo reference="esp32">
-                <mu1>1.0</mu1>
-                <mu2>1.0</mu2>
-            </gazebo>
-        </xacro:if>
+        <xacro:esp32_unit suffix="" parent="esp32_adapter"
+            rpy="${pi} 0 ${-pi_2}" x="0.002" y="0" z="-0.01"/>
     </xacro:unless>
     <!-- .......................... LIDAR spacers .......................... -->
@@ -438,11 +264,5 @@
         <origin xyz="${-0.0575} -0.0035 0.0125" rpy="0 0 0"/>
     </joint>
-    <xacro:if value="${gazebo}">
-        <gazebo reference="ld19">
-            <selfCollide>false</selfCollide>
-            <mu1 value="0.05" />
-            <mu2 value="0.05" />
-        </gazebo>
-    </xacro:if>
+    <xacro:gazebo_friction_sensor link="ld19" mu1="0.05" mu2="0.05"/>
     <link name="laser_scan"/>
     <joint name="laser_joint" type="fixed">
@@ -482,10 +302,5 @@
             <origin xyz="-0.03 0.025 0.0025" rpy="0 0 0"/>
         </joint>
-        <xacro:if value="${gazebo}">
-            <gazebo reference="lidar_serial">
-                <mu1>1.0</mu1>
-                <mu2>1.0</mu2>
-            </gazebo>
-        </xacro:if>
+        <xacro:gazebo_friction link="lidar_serial"/>
     </xacro:unless>
         <!-- ....................... Servo Definitions ........................ -->
@@ -553,10 +368,5 @@
             <origin xyz="-0.02 0 0.025" rpy="0 0 0"/>
         </joint>
-        <xacro:if value="${gazebo}">
-            <gazebo reference="stereo">
-                <mu1>1.0</mu1>
-                <mu2>1.0</mu2>
-            </gazebo>
-        </xacro:if>
+        <xacro:gazebo_friction link="stereo"/>
         <!-- ........................ Wall definitions ...................... -->
         <xacro:complete_lateral_wall id="curve" parent="base_l2_s1" side="1"
@@ -603,10 +413,5 @@
             <origin xyz="0 0.0335 0.0125" rpy="0 0 0"/>
         </joint>
-        <xacro:if value="${gazebo}">
-            <gazebo reference="${rasp}">
-                <mu1>1.0</mu1>
-                <mu2>1.0</mu2>
-            </gazebo>
-        </xacro:if>
+        <xacro:gazebo_friction link="${rasp}"/>
         <!-- .......................... Microphone .................................. -->
         <link name="microphone">
@@ -639,10 +444,5 @@
             <origin xyz="-0.0275 0.0 0.06" rpy="0 0 0"/>
         </joint>
-        <xacro:if value="${gazebo}">
-            <gazebo reference="microphone">
-                <mu1>1.0</mu1>
-                <mu2>1.0</mu2>
-            </gazebo>
-        </xacro:if>
+        <xacro:gazebo_friction link="microphone"/>
     </xacro:unless>
     <!-- ........................ Touch sensors ........................ -->
@@ -670,75 +470,9 @@
         offset_x="${0.0577/2}" offset_y="${0.0607/2}" x="0.004" y="0" z="0.0025"/>
         <!-- .......................... Esp32 Adapter ....................... -->
-        <link name="esp32_2_adapter">
-            <visual>
-                <origin xyz="0 0 0" rpy="0 0 0"/>
-                <geometry>
-                    <mesh filename="package://orion_description/meshes/esp32_adp.stl"
-                    scale="0.001 0.001 0.001"/>
-                </geometry>
-                <material name="RaspberryGreen"/>
-            </visual>
-            <collision>
-                <origin xyz="0 0 0" rpy="0 0 0"/>
-                <geometry>
-                    <mesh filename="package://orion_description/meshes/esp32_adp.stl"
-                    scale="0.001 0.001 0.001"/>
-                </geometry>
-            </collision>
-            <inertial>
-                <origin xyz="0 0 0" rpy="0 0 0"/>
-                <mass value="0.030"/>
-                <inertia ixx="1.1184306270694732e-05" ixy="0.0" ixz="0.0"
-                iyy="1.021680627069473e-05" iyz="0.0"
-                izz="2.0812499999999994e-05"/>
-            </inertial>
-        </link>
-        <joint name="esp32_2_adapter_joint" type="fixed">
-            <parent link="base_l3_s1"/>
-            <child link="esp32_2_adapter"/>
-            <origin xyz="0.004 0 0.0125" rpy="0 0 0"/>
-        </joint>
-        <xacro:if value="${gazebo}">
-            <gazebo reference="esp32_2_adapter">
-                <mu1>1.0</mu1>
-                <mu2>1.0</mu2>
-            </gazebo>
-        </xacro:if>
+        <xacro:esp32_adapter_unit suffix="_2" parent="base_l3_s1"
+            rpy="0 0 0" x="0.004" y="0" z="0.0125"/>
         <!-- ....................... ESP32 ....................................... -->
-        <link name="esp32_2">
-            <visual>
-                <origin xyz="0 0 0" rpy="0 0 ${-pi_2}"/>
-                <geometry>
-                    <mesh filename="package://orion_description/meshes/esp32.stl"
-                    scale="0.001 0.001 0.001"/>
-                </geometry>
-                <material name="SoftBlack"/>
-            </visual>
-            <collision>
-                <origin xyz="0 0 0" rpy="0 0 ${-pi_2}"/>
-                <geometry>
-                    <mesh filename="package://orion_description/meshes/esp32.stl"
-                    scale="0.001 0.001 0.001"/>
-                </geometry>
-            </collision>
-            <inertial>
-                <origin xyz="0 0 0" rpy="0 0 ${-pi_2}"/>
-                <mass value="0.0201"/>
-                <inertia ixx="4.904162034278915e-06" ixy="0.0" ixz="0.0"
-                iyy="1.5830928543782435e-06" iyz="0.0"
-                izz="6.0040505352397235e-06"/>
-            </inertial>
-        </link>
-        <joint name="esp32_2_joint" type="fixed">
-            <parent link="esp32_2_adapter"/>
-            <child link="esp32_2"/>
-            <origin xyz="0.002 0 0.01" rpy="0 0 0"/>
-        </joint>
-        <xacro:if value="${gazebo}">
-            <gazebo reference="esp32_2">
-                <mu1>1.0</mu1>
-                <mu2>1.0</mu2>
-            </gazebo>
-        </xacro:if>
+        <xacro:esp32_unit suffix="_2" parent="esp32_2_adapter"
+            rpy="0 0 ${-pi_2}" x="0.002" y="0" z="0.01"/>
     </xacro:unless>
     <!-- .......................... Screen Sup ................................ -->
@@ -750,16 +484,5 @@
             scale="0.001 0.001 0.001"/>
         </geometry>
-        <xacro:if value="${color == 'mdf'}">
-            <material name="MDF"/>
-        </xacro:if>
-        <xacro:if value="${color == 'transparent'}">
-            <material name="TransparentBlack"/>
-        </xacro:if>
-        <xacro:if value="${color == 'pla'}">
-            <material name="PLAWhite"/>
-        </xacro:if>
-        <xacro:if value="${color == 'gold'}">
-            <material name="Gold"/>
-        </xacro:if>
+        <xacro:apply_color_material/>
     </visual>
     <collision>
@@ -783,10 +506,5 @@
         <origin xyz="0 0 0" rpy="0 0 0"/>
     </joint>
-    <xacro:if value="${gazebo}">
-        <gazebo reference="screen_sup">
-            <mu1>1.0</mu1>
-            <mu2>1.0</mu2>
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