Commit message: Description: Replacing color and gz friction with macros, clearning macro files and updating comments

File: orion_description/urdf/include/orion_macros.urdf.xacro (robot description, xacro)
@@ -10,4 +10,37 @@
     <xacro:property name="pi_6" value="${pi / 6}"/>
     <xacro:property name="pi_8" value="${pi / 8}"/>
+    <!--/////////////////// GAZEBO FRICTION MACROS //////////////////////-->
+    <!-- Standard Coulomb friction tags emitted only when ${gazebo} is true.
+         Defaults match the most common case (mu1=mu2=1.0). -->
+    <xacro:macro name="gazebo_friction" params="link mu1:=1.0 mu2:=1.0">
+        <xacro:if value="${gazebo}">
+            <gazebo reference="${link}">
+                <mu1>${mu1}</mu1>
+                <mu2>${mu2}</mu2>
+            </gazebo>
+        </xacro:if>
+    </xacro:macro>
+    <!-- Friction + contact stiffness (kp) and damping (kd). Used for rolling
+         contacts (caster wheel/middle) where contact dynamics matter. -->
+    <xacro:macro name="gazebo_friction_contact" params="link mu1 mu2 kp kd">
+        <xacro:if value="${gazebo}">
+            <gazebo reference="${link}">
+                <mu1>${mu1}</mu1>
+                <mu2>${mu2}</mu2>
+                <kp>${kp}</kp>
+                <kd>${kd}</kd>
+            </gazebo>
+        </xacro:if>
+    </xacro:macro>
+    <!-- Friction for sensor links that should not self-collide. -->
+    <xacro:macro name="gazebo_friction_sensor" params="link mu1:=0.05 mu2:=0.05">
+        <xacro:if value="${gazebo}">
+            <gazebo reference="${link}">
+                <selfCollide>false</selfCollide>
+                <mu1>${mu1}</mu1>
+                <mu2>${mu2}</mu2>
+            </gazebo>
+        </xacro:if>
+    </xacro:macro>
     <!--///////////////////// 10 x 80 SPACERS MACROS ///////////////////////-->
     <!-- ......................... Single custom spacer ................... -->
@@ -62,10 +95,5 @@
             <origin xyz="${x*mulf} ${y*muls} ${z+0.0025}" rpy="0 0 0"/>
         </joint>
-        <xacro:if value="${gazebo}">
-        <gazebo reference="spacer_l${level}_${front}${side}">
-            <mu1>1.0</mu1>
-            <mu2>1.0</mu2>
-        </gazebo>
-    </xacro:if>
+        <xacro:gazebo_friction link="spacer_l${level}_${front}${side}"/>
     </xacro:macro>
     <!-- ....................... Double 10x80 Spacer .................... -->
@@ -90,16 +118,5 @@
                 scale="0.001 0.001 0.001"/>
             </geometry>
-            <xacro:if value="${color == 'mdf'}">
-                <material name="MDF"/>
-            </xacro:if>
-            <xacro:if value="${color == 'transparent'}">
-                <material name="TransparentBlack"/>
-            </xacro:if>
-            <xacro:if value="${color == 'pla'}">
-                <material name="PLAWhite"/>
-            </xacro:if>
-            <xacro:if value="${color == 'gold'}">
-                <material name="Gold"/>
-            </xacro:if>
+            <xacro:apply_color_material/>
         </visual>
         <collision>
@@ -123,10 +140,5 @@
             <origin xyz="${x + (mul*0.115/2)} ${y} ${z}" rpy="0 0 0"/>
         </joint>
-        <xacro:if value="${gazebo}">
-        <gazebo reference="base_l${level}_s${side}">
-            <mu1>1.0</mu1>
-            <mu2>1.0</mu2>
-        </gazebo>
-        </xacro:if>
+        <xacro:gazebo_friction link="base_l${level}_s${side}"/>
     </xacro:macro>
     <!-- ...................... Complete base ............................ -->
@@ -181,8 +193,5 @@
             <origin xyz="${x*mulf} ${y*muls} ${z+0.0025}" rpy="0 0 0"/>
         </joint>
-        <gazebo reference="motor_support_${front}${side}">
-            <mu1>1.0</mu1>
-            <mu2>1.0</mu2>
-        </gazebo>
+        <xacro:gazebo_friction link="motor_support_${front}${side}"/>
         <!-- Link motor dc definition-->
         <link name="motor_dc_${front}${side}">
@@ -215,8 +224,5 @@
             <origin xyz="0 ${-0.05625*muls} 0" rpy="0 0 0"/>
         </joint>
-        <gazebo reference="motor_dc_${front}${side}">
-            <mu1>1.0</mu1>
-            <mu2>1.0</mu2>
-        </gazebo>
+        <xacro:gazebo_friction link="motor_dc_${front}${side}"/>
         <!-- Coupling definition-->
         <link name="coupling_${front}${side}">
@@ -244,4 +250,17 @@
         </inertial>
         </link>
+        <!-- NOTE: The coupling link is the rotating member that acts as the
+             "wheel joint" for ros2_control / diff_drive_controller. The actual
+             rubber tire (neumatic) and stop ring are rigidly attached to it via
+             fixed joints. Using coupling as the rotational element preserves the
+             mechanical chain (motor shaft -> coupling -> ring -> tire) so the
+             dynamics stay physically faithful. -->
+        <!-- Joint limits derived from motor nominal specs at 12V (no load):
+               1000 RPM motor -> 1000 * 2*pi/60 ~= 104.72 rad/s, effort 0.01079 N*m
+                100 RPM motor ->  100 * 2*pi/60 ~=  10.47 rad/s, effort 0.08336 N*m
+             Linear velocity at wheel_radius=0.033675 m (see
+             orion_control/config/mobile_base_controller.yaml). The
+             ros2_control command_interface limits are intentionally lower
+             (see orion_ros2_control.urdf.xacro for the conservative cap). -->
         <joint name="coupling_${front}${side}_joint" type="continuous">
             <axis xyz="0.0 0.0 1.0"/>
@@ -256,8 +275,5 @@
             <origin xyz="0 ${(0.01120 + 0.000325)*muls} 0" rpy="${-pi_2*muls+orin} 0 0"/>
         </joint>
-        <gazebo reference="coupling_${front}${side}">
-            <mu1>1.0</mu1>
-            <mu2>1.0</mu2>
-        </gazebo>
+        <xacro:gazebo_friction link="coupling_${front}${side}"/>
         <!-- Ring definition -->
         <link name="ring_${front}${side}">
@@ -290,8 +306,5 @@
             <origin xyz="0 0 ${0.0068*muls}" rpy="0 0 0"/>
         </joint>
-        <gazebo reference="ring_${front}${side}">
-            <mu1>1.0</mu1>
-            <mu2>1.0</mu2>
-        </gazebo>
+        <xacro:gazebo_friction link="ring_${front}${side}"/>
         <!-- Neumatic definition-->
         <link name="neumatic_${front}${side}">
@@ -325,8 +338,5 @@
             <origin xyz="0 0 0" rpy="0 0 0"/>
         </joint>
-        <gazebo reference="neumatic_${front}${side}">
-            <mu1>1.0</mu1>
-            <mu2>0.8</mu2>
-        </gazebo>
+        <xacro:gazebo_friction link="neumatic_${front}${side}" mu1="1.0" mu2="0.8"/>
     </xacro:macro>
     <!--////////////////////////// CASTER WHEEL ////////////////////////////-->
@@ -367,8 +377,5 @@
             <origin xyz="${x} ${y} ${z}" rpy="0 0 0"/>
         </joint>
-        <gazebo reference="caster_base_${front}">
-            <mu1>1.0</mu1>
-            <mu2>1.0</mu2>
-        </gazebo>
+        <xacro:gazebo_friction link="caster_base_${front}"/>
         <!-- Caster middle definition-->
         <link name="caster_middle_${front}">
@@ -403,10 +410,6 @@
             <dynamics damping="0.05" friction="0.0"/>
         </joint>
-        <gazebo reference="caster_middle_${front}">
-            <mu1>0.01</mu1>
-            <mu2>0.01</mu2>
-            <kp>100000.0</kp>
-            <kd>10.0</kd>
-        </gazebo>
+        <xacro:gazebo_friction_contact link="caster_middle_${front}"
+            mu1="0.01" mu2="0.01" kp="100000.0" kd="10.0"/>
         <!-- Caster wheel definition-->
         <link name="caster_wheel_${front}">
@@ -441,10 +444,6 @@
             <dynamics damping="0.05" friction="0.0"/>
         </joint>
-        <gazebo reference="caster_wheel_${front}">
-            <mu1>0.01</mu1>
-            <mu2>0.01</mu2>
-            <kp>100000.0</kp>
-            <kd>10.0</kd>
-        </gazebo>
+        <xacro:gazebo_friction_contact link="caster_wheel_${front}"
+            mu1="0.01" mu2="0.01" kp="100000.0" kd="10.0"/>
     </xacro:macro>
     <!-- ///////////////////// BATTERIES MACROS ////////////////////////////-->
@@ -490,8 +489,5 @@
             <origin xyz="${x*inv} ${y} ${z}" rpy="0 0 0"/>
         </joint>
-        <gazebo reference="${element}_${num}">
-            <mu1>1.0</mu1>
-            <mu2>1.0</mu2>
-        </gazebo>
+        <xacro:gazebo_friction link="${element}_${num}"/>
     </xacro:macro>
     <!-- ........................ Battery holder macro ........................ -->
@@ -527,8 +523,5 @@
             <origin xyz="${x} ${y} ${z}" rpy="0 0 0"/>
         </joint>
-        <gazebo reference="${element}_${num}">
-            <mu1>1.0</mu1>
-            <mu2>1.0</mu2>
-        </gazebo>
+        <xacro:gazebo_friction link="${element}_${num}"/>
     </xacro:macro>
     <xacro:macro name="stack_bat" params="parent num x y z">
@@ -581,8 +574,5 @@
             <origin xyz="${x} ${y*inv} ${z}" rpy="0 0 0"/>
         </joint>
-        <gazebo reference="servo_support_${side}">
-            <mu1>1.0</mu1>
-            <mu2>1.0</mu2>
-        </gazebo>
+        <xacro:gazebo_friction link="servo_support_${side}"/>
         <!-- Servo Link -->
         <link name="servo_${side}">
@@ -615,8 +605,5 @@
             <origin xyz="0 ${-0.0216*inv} -0.01375" rpy="0 0 0"/>
         </joint>
-        <gazebo reference="servo_${side}">
-            <mu1>0.05</mu1>
-            <mu2>0.05</mu2>
-        </gazebo>
+        <xacro:gazebo_friction link="servo_${side}" mu1="0.05" mu2="0.05"/>
         <!-- Servo Conn -->
         <link name="servo_conn_${side}">
@@ -652,8 +639,5 @@
             <dynamics damping="0.05" friction="0.002"/>
         </joint>
-        <gazebo reference="servo_conn_${side}">
-            <mu1>0.05</mu1>
-            <mu2>0.05</mu2>
-        </gazebo>
+        <xacro:gazebo_friction link="servo_conn_${side}" mu1="0.05" mu2="0.05"/>
     </xacro:macro>
     <!--///////////////////// SPEAKERS MACROS ///////////////////////-->
@@ -701,8 +685,5 @@
             <origin xyz="${x*mulf} ${y*muls} ${z}" rpy="0 0 0"/>
         </joint>
-        <gazebo reference="speaker_sup_${front}${side}">
-            <mu1>1.0</mu1>
-            <mu2>1.0</mu2>
-        </gazebo>
+        <xacro:gazebo_friction link="speaker_sup_${front}${side}"/>
         <!-- Speaker -->
         <link name="speaker_${front}${side}">
@@ -735,8 +716,5 @@
             <origin xyz="0 ${0.0375*muls/2} 0" rpy="0 0 0"/>
         </joint>
-        <gazebo reference="speaker_${front}${side}">
-            <mu1>1.0</mu1>
-            <mu2>1.0</mu2>
-        </gazebo>
+        <xacro:gazebo_friction link="speaker_${front}${side}"/>
     </xacro:macro>
     <!-- ///////////////////////////// WALL MACROS //////////////////////// -->
@@ -754,16 +732,5 @@
                 scale="0.001 0.001 0.001"/>
             </geometry>
-            <xacro:if value="${color == 'mdf'}">
-                <material name="MDF"/>
-            </xacro:if>
-            <xacro:if value="${color == 'transparent'}">
-                <material name="TransparentBlack"/>
-            </xacro:if>
-            <xacro:if value="${color == 'pla'}">
-                <material name="PLAWhite"/>
-            </xacro:if>
-            <xacro:if value="${color == 'gold'}">
-                <material name="Gold"/>
-            </xacro:if>
+            <xacro:apply_color_material/>
         </visual>
         <collision>
@@ -787,8 +754,6 @@
         <origin xyz="${x} ${(y+0.00075)*muls} ${z}" rpy="0 0 0"/>
         </joint>
-        <gazebo reference="wall_${id}_${level}_${side}">
-            <mu1>0.05</mu1>
-            <mu2>0.05</mu2>
-        </gazebo>
+        <xacro:gazebo_friction link="wall_${id}_${level}_${side}"
+            mu1="0.05" mu2="0.05"/>
     </xacro:macro>
     <xacro:macro name="complete_front_wall"
@@ -808,16 +773,5 @@
                 scale="0.001 0.001 0.001"/>
             </geometry>
-            <xacro:if value="${color == 'mdf'}">
-                <material name="MDF"/>
-            </xacro:if>
-            <xacro:if value="${color == 'transparent'}">
-                <material name="TransparentBlack"/>
-            </xacro:if>
-            <xacro:if value="${color == 'pla'}">
-                <material name="PLAWhite"/>
-            </xacro:if>
-            <xacro:if value="${color == 'gold'}">
-                <material name="Gold"/>
-            </xacro:if>
+            <xacro:apply_color_material/>
         </visual>
         <collision>
@@ -841,8 +795,5 @@
         <origin xyz="${(x+0.00075)*mulf} 0 ${z}" rpy="0 0 0"/>
         </joint>
-        <gazebo reference="wall_${id}_${level}_${front}">
-            <mu1>1.0</mu1>
-            <mu2>1.0</mu2>
-        </gazebo>
+        <xacro:gazebo_friction link="wall_${id}_${level}_${front}"/>
     </xacro:macro>
     <!-- /////////////////////////// Generic Metric Spacer /////////////////-->
@@ -894,9 +845,5 @@
             <origin xyz="${x} ${y} ${z}" rpy="0 0 0"/>
         </joint>
-        <!-- Gazebo Spacer -->
-        <gazebo reference="${id}_${element}_${front}${side}">
-            <mu1>1.0</mu1>
-            <mu2>1.0</mu2>
-        </gazebo>
+        <xacro:gazebo_friction link="${id}_${element}_${front}${side}"/>
     </xacro:macro>
     <!-- 2 symetric hex spacers by considering offset -->
@@ -988,10 +935,5 @@
             <child link="touch_sensor_${prefix}${side}"/>
         </joint>
-        <xacro:if value="${gazebo}">
-            <gazebo reference="touch_sensor_${prefix}${side}">
-                <mu1>1.0</mu1>
-                <mu2>1.0</mu2>
-            </gazebo>
-        </xacro:if>
+        <xacro:gazebo_friction link="touch_sensor_${prefix}${side}"/>
         <xacro:property name="rotR" value="0"/>
         <xacro:property name="rotP" value="0"/>
@@ -1019,16 +961,5 @@
                     scale="0.001 0.001 0.001"/>
                 </geometry>
-                <xacro:if value="${color == 'mdf'}">
-                    <material name="MDF"/>
-                </xacro:if>
-                <xacro:if value="${color == 'transparent'}">
-                    <material name="TransparentBlack"/>
-                </xacro:if>
-                <xacro:if value="${color == 'pla'}">
-                    <material name="PLAWhite"/>
-                </xacro:if>
-                <xacro:if value="${color == 'gold'}">
-                    <material name="Gold"/>
-                </xacro:if>
+                <xacro:apply_color_material/>
             </visual>
             <collision>
@@ -1052,10 +983,5 @@
             <child link="touch_sup_${prefix}${side}"/>
         </joint>
-        <xacro:if value="${gazebo}">
-            <gazebo reference="touch_sup_${prefix}${side}">
-                <mu1>1.0</mu1>
-                <mu2>1.0</mu2>
-            </gazebo>
-        </xacro:if>
+        <xacro:gazebo_friction link="touch_sup_${prefix}${side}"/>
     </xacro:macro>
     <!-- /////////////////////// Cameras macros //////////////////////// -->
@@ -1075,3 +1001,110 @@
         </joint>
     </xacro:macro>
+    <!--//////////////// COMPOSITE / REPEATED UNITS //////////////////////-->
+    <!-- Battery holder platform unit. Suffix is empty for the first instance
+         (link "bat_platform") and "_2" for the second ("bat_platform_2") to
+         preserve the existing parent references used by stack_bat calls. -->
+    <xacro:macro name="bat_platform_unit" params="suffix parent x y z">
+        <link name="bat_platform${suffix}">
+            <visual>
+                <origin xyz="0 0 0" rpy="0 0 ${pi_2}"/>
+                <geometry>
+                    <mesh filename="package://orion_description/meshes/bathold_support.stl"
+                        scale="0.001 0.001 0.001"/>
+                </geometry>
+                <xacro:apply_color_material/>
+            </visual>
+            <collision>
+                <origin xyz="0 0 0" rpy="0 0 ${pi_2}"/>
+                <geometry>
+                    <mesh filename="package://orion_description/meshes/bathold_support.stl"
+                        scale="0.001 0.001 0.001"/>
+                </geometry>
+            </collision>
+            <inertial>
+                <origin xyz="0 0 0" rpy="0 0 ${pi_2}"/>
+                <mass value="0.018"/>
+                <inertia ixx="1.2564374999999998e-05" ixy="0.0" ixz="0.0"
+                        iyy="2.6539499999999996e-05" iyz="0.0"
+                        izz="3.9091874999999996e-05"/>
+            </inertial>
+        </link>
+        <joint name="bat_platform${suffix}_joint" type="fixed">
+            <parent link="${parent}"/>
+            <child link="bat_platform${suffix}"/>
+            <origin xyz="${x} ${y} ${z}" rpy="0 0 0"/>
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
File: orion_description/urdf/include/orion_materials.urdf.xacro (robot description, xacro)
@@ -51,3 +51,19 @@
         <color rgba="0.72 0.52 0.35 1.0"/>
     </material>
+    <!-- Selects the visual material for structural panels based on the global
+         ${color} property. Supported values: 'mdf', 'transparent', 'pla', 'gold'. -->
+    <xacro:macro name="apply_color_material">
+        <xacro:if value="${color == 'mdf'}">
+            <material name="MDF"/>
+        </xacro:if>
+        <xacro:if value="${color == 'transparent'}">
+            <material name="TransparentBlack"/>
+        </xacro:if>
+        <xacro:if value="${color == 'pla'}">
+            <material name="PLAWhite"/>
+        </xacro:if>
+        <xacro:if value="${color == 'gold'}">
+            <material name="Gold"/>
+        </xacro:if>
+    </xacro:macro>
 </robot>

File: orion_description/urdf/include/orion_ros2_control.urdf.xacro (robot description, xacro)
@@ -2,5 +2,10 @@
 <!-- @file orion_ros2_control.urdf.xacro
      @brief ros2_control hardware interface tags for ORION differential drive and servo arms.
-     Exposes DiffDriveOrion and ForwardOrion plugins to the controller manager. -->
+     Exposes DiffDriveOrion and ForwardOrion plugins to the controller manager.
+     NOTE on naming: `coupling_11_joint` / `coupling_12_joint` are the rotating
+     joints that physically act as the differential-drive wheel joints. The
+     URDF chain is motor_shaft -> coupling (continuous) -> ring (fixed) ->
+     neumatic / tire (fixed). The coupling is treated as the wheel joint to
+     keep the mechanical chain physically faithful to the real hardware. -->
 <robot xmlns:xacro="http://www.ros.org/wiki/xacro">
     <xacro:if value="${ros2_control}">

File: orion_description/urdf/orion.urdf.xacro (robot description, xacro)
@@ -2,8 +2,21 @@
 <!-- @file orion.urdf.xacro
      @brief Top-level robot description for ORION. Declares all configurable
-     properties (camera, servo, rasp, motor, ctl_type, etc.) and includes
+     arguments (camera, servo, rasp, motor, ctl_type, color, etc.) and includes
      the modular xacro files for materials, macros, base, arms, cameras,
      and ros2_control tags. -->
 <robot xmlns:xacro="http://www.ros.org/wiki/xacro" name="orion">
+    <!-- Configurable arguments. Defaults allow standalone xacro processing
+         (e.g. `xacro orion.urdf.xacro`) without requiring every value to be
+         passed from a launch file. -->
+    <xacro:arg name="camera" default="os30a"/>
+    <xacro:arg name="servo" default="true"/>
+    <xacro:arg name="g_mov" default="false"/>
+    <xacro:arg name="rasp" default="rpi5"/>
+    <xacro:arg name="gazebo" default="false"/>
+    <xacro:arg name="ros2_control" default="false"/>
+    <xacro:arg name="simplified" default="false"/>
+    <xacro:arg name="motor" default="100"/>
+    <xacro:arg name="ctl_type" default="micro_ros"/>
+    <xacro:arg name="color" default="gold"/>
     <xacro:property name="camera" default="$(arg camera)"/>
     <xacro:property name="servo" default="$(arg servo)"/>
@@ -13,8 +26,8 @@
     <xacro:property name="ros2_control" default="$(arg ros2_control)"/>
     <xacro:property name="simplified" default="$(arg simplified)"/>
-    <xacro:property name="motor" value="$(arg motor)"/>
+    <xacro:property name="motor" default="$(arg motor)"/>
     <xacro:property name="ctl_type" default="$(arg ctl_type)"/>
-    <!-- For colors consider mdf, transparent or pla -->
-    <xacro:property name="color" default="gold"/>
+    <!-- Visual color for structural panels: 'mdf', 'transparent', 'pla', 'gold' -->
+    <xacro:property name="color" default="$(arg color)"/>
     <!-- Include other files -->
     <xacro:include filename="$(find orion_description)/urdf/include/orion_materials.urdf.xacro"/>
