Commit message: Assets: Updating ORION partial assembly | Control/Description: Updating servo connector name

File: orion_description/urdf/include/orion_macros.urdf.xacro (robot description, xacro)
@@ -631,5 +631,5 @@
         </inertial>
         </link>
-        <joint name="servo_conn${side}_joint" type="revolute">
+        <joint name="servo_conn_${side}_joint" type="revolute">
             <axis xyz="0.0 0.0 1.0"/>
             <parent link="servo_${side}"/>

File: orion_description/urdf/include/orion_ros2_control.urdf.xacro (robot description, xacro)
@@ -52,7 +52,7 @@
                         <param name="feedback_topic">fwd_servo_left_feedback</param>
                         <param name="cmd_topic">fwd_servo_left_cmd</param>
-                        <param name="servo_name">servo_conn1_joint</param>
+                        <param name="servo_name">servo_conn_1_joint</param>
                     </hardware>
-                    <joint name="servo_conn1_joint">
+                    <joint name="servo_conn_1_joint">
                         <command_interface name="position" />
                         <state_interface name="position" />
@@ -64,7 +64,7 @@
                         <param name="feedback_topic">fwd_servo_right_feedback</param>
                         <param name="cmd_topic">fwd_servo_right_cmd</param>
-                        <param name="servo_name">servo_conn2_joint</param>
+                        <param name="servo_name">servo_conn_2_joint</param>
                     </hardware>
-                    <joint name="servo_conn2_joint">
+                    <joint name="servo_conn_2_joint">
                         <command_interface name="position" />
                         <state_interface name="position" />
