Commit message: Description: Adding meshes and xacro for g_mov as it is no longer maintained, updated camera links

File: orion_description/urdf/include/orion_cameras.urdf.xacro (robot description, xacro)
@@ -169,9 +169,10 @@
             <origin xyz="0 0 -0.0205" rpy="0 0 0"/>
         </joint>
-        <!-- ......................... Usage of GMov ...................................  -->
+        <!-- ......................... Usage of G Mov ...................................  -->
+        <!-- G Mov module macros are defined in orion_g_mov.urdf.xacro and
+             included at the top level of orion.urdf.xacro. -->
         <xacro:if value="${g_mov}">
-            <xacro:include filename="$(find g_mov_description)/urdf/g_mov_macros.urdf.xacro"/>
             <xacro:g_mov_assem parent="${level_cam}" spacer="m3x10" offset="${0.033/2}"
-                x="0.013825" y="0.035" z="0.0025" joint_prefix="g_mov"/>
+                x="0.013825" y="0.035" z="0.0025"/>
         </xacro:if>
         <!-- ......................... Camera sensors links ............................ -->

File: orion_description/urdf/include/orion_macros.urdf.xacro (robot description, xacro)
@@ -831,4 +831,10 @@
                         izz="4.443388969597693e-09"/>
             </xacro:if>
+            <xacro:if value="${id == 'm3x15'}">
+                <mass value="0.0017"/>
+                <inertia ixx="5.2825999244689955e-08" ixy="0" ixz="0"
+                        iyy="5.4441082699086494e-08" iyz="0"
+                        izz="9.66508345439654e-09"/>
+            </xacro:if>
             <xacro:if value="${id == 'm3x20'}">
                 <mass value="0.0024"/>
@@ -836,4 +842,14 @@
                         iyy="8.648216387229408e-08" iyz="0"
                         izz="1.333016690879308e-08"/>
+            </xacro:if>
+            <!-- NOTE: m3x6 iyy value reconstructed from a corrupted source
+                 ('.272650140158067e-09'); leading digit was missing. Picked
+                 4.272...e-09 based on the ixx/iyy ratio pattern of larger
+                 spacers (~1.05x for short ones). Verify if precision matters. -->
+            <xacro:if value="${id == 'm3x6'}">
+                <mass value="0.00072"/>
+                <inertia ixx="3.9036000675201425e-09" ixy="0" ixz="0"
+                        iyy="4.272650140158067e-09" iyz="0"
+                        izz="3.9990500726379235e-09"/>
             </xacro:if>
         </inertial>

File: orion_description/urdf/orion.urdf.xacro (robot description, xacro)
@@ -33,4 +33,5 @@
     <xacro:include filename="$(find orion_description)/urdf/include/orion_materials.urdf.xacro"/>
     <xacro:include filename="$(find orion_description)/urdf/include/orion_macros.urdf.xacro"/>
+    <xacro:include filename="$(find orion_description)/urdf/include/orion_g_mov.urdf.xacro"/>
     <xacro:include filename="$(find orion_description)/urdf/include/orion_base.urdf.xacro"/>
     <xacro:include filename="$(find orion_description)/urdf/include/orion_arms.urdf.xacro"/>
