Commit message: Base: Fix servo orientation | Control: Updating params | Utils: Adding pending node

File: orion_description/urdf/include/orion_ros2_control.urdf.xacro (robot description, xacro)
@@ -8,4 +8,7 @@
                     <param name="left_wheel_name">coupling_11_joint</param>
                     <param name="right_wheel_name">coupling_12_joint</param>
+                    <param name="motor_cmd_topic">/diff_ctl_motor_cmd</param>
+                    <param name="left_enc_topic">/diff_ctl_left_enc</param>
+                    <param name="right_enc_topic">/diff_ctl_right_enc</param>
                     <xacro:if value="${motor == 1000}">
                         <param name="enc_ticks_per_rev">204</param>

File: orion_description/urdf/orion.urdf.xacro (robot description, xacro)
@@ -9,7 +9,7 @@
     <xacro:property name="simplified" default="$(arg simplified)"/>
     <xacro:property name="motor" value="$(arg motor)"/>
-    <xacro:property name="ctl_type" default="micro_ros"/>
+    <xacro:property name="ctl_type" default="$(arg ctl_type)"/>
     <!-- For colors consider mdf, transparent or pla -->
-    <xacro:property name="color" default="pla"/>
+    <xacro:property name="color" default="gold"/>
     <!-- Include other files -->
     <xacro:include filename="$(find orion_description)/urdf/include/orion_materials.urdf.xacro"/>

Commit message: Description: Updating g_mov module | Utils Py: Adding accelerometer and servo scripts | Bringup: Updating controller call for g_mov servo

File: orion_description/urdf/include/orion_ros2_control.urdf.xacro (robot description, xacro)
@@ -72,4 +72,18 @@
                 </ros2_control>
             </xacro:if>
+            <xacro:if value="${g_mov}">
+                <ros2_control name="FwdGMovRealRobot" type="system">
+                    <hardware>
+                        <plugin>orion_control/ForwardOrion</plugin>
+                        <param name="feedback_topic">fwd_servo_g_mov_feedback</param>
+                        <param name="cmd_topic">fwd_servo_g_mov_cmd</param>
+                        <param name="servo_name">g_mov_servo_conn_joint</param>
+                    </hardware>
+                    <joint name="g_mov_servo_conn_joint">
+                        <command_interface name="position" />
+                        <state_interface name="position" />
+                    </joint>
+                </ros2_control>
+            </xacro:if>
         </xacro:if>
     </xacro:if>
