Commit message: General: Updating formatting and comments on codes, review of modifications

File: orion_description/urdf/include/orion_base.urdf.xacro (robot description, xacro)
@@ -509,5 +509,5 @@
     <!-- ...................... Screen ................................. -->
     <link name="screen">
-    <visual>
+    <visual name="screen">
         <origin xyz="0 0 0" rpy="${pi_4} 0 ${pi_2}"/>
         <geometry>

File: orion_description/urdf/orion.urdf.xacro (robot description, xacro)
@@ -6,7 +6,5 @@
      and ros2_control tags. -->
 <robot xmlns:xacro="http://www.ros.org/wiki/xacro" name="orion">
-    <!-- Configurable arguments. Defaults allow standalone xacro processing
-         (e.g. `xacro orion.urdf.xacro`) without requiring every value to be
-         passed from a launch file. -->
+    <!-- Configurable arguments -->
     <xacro:arg name="camera" default="os30a"/>
     <xacro:arg name="servo" default="true"/>
@@ -30,5 +28,5 @@
     <!-- Visual color for structural panels: 'mdf', 'transparent', 'pla', 'gold' -->
     <xacro:property name="color" default="$(arg color)"/>
-    <!-- Include other files -->
+    <!-- Include other files for robot description -->
     <xacro:include filename="$(find orion_description)/urdf/include/orion_materials.urdf.xacro"/>
     <xacro:include filename="$(find orion_description)/urdf/include/orion_macros.urdf.xacro"/>
